Commit message: correct the limit of actual movement speed/update the correct urdf file

File: resources/robots/astra/astra.urdf (robot description, URDF)
Before this commit: robot ASTRA_Sim_Simplified, 16 links, 15 joints
Links:
- removed link Dummy_link
- removed link SPINE_BASE
- removed link backbase
- removed link frontbase
- added link Backpart, mass 2.332620946077069; collision mesh filename=meshes/Backpart.stl scale=0.001 0.001 0.001; visual mesh filename=meshes/Backpart.stl scale=0.001 0.001 0.001
- added link Base_link, mass 0.0036615962412117928; collision mesh filename=meshes/Base_link.stl scale=0.001 0.001 0.001; visual mesh filename=meshes/Base_link.stl scale=0.001 0.001 0.001
- added link Frontpart, mass 2.6950744218640232; collision mesh filename=meshes/Frontpart.stl scale=0.001 0.001 0.001; visual mesh filename=meshes/Frontpart.stl scale=0.001 0.001 0.001
- added link Spine, mass 0.2716788388343432; collision mesh filename=meshes/Spine.stl scale=0.001 0.001 0.001; visual mesh filename=meshes/Spine.stl scale=0.001 0.001 0.001
Joints:
- removed joint Dummy_link_Back_k_DU
- removed joint SPINE_BASE_DU_k_Base
- removed joint backbase_RL_j_hip
- removed joint backbase_RR_j_hip
- removed joint frontbase_FL_j_hip
- removed joint frontbase_FR__j_hip
- removed joint frontbase_F_j_spine
- added joint Backpart_RL_j_hip: type revolute, parent Backpart, child RL_hip, origin xyz=-0.17573185000000002 0.0706705 -0.0175 rpy=-1.5707963267948968 7.689375450873787e-28 -3.1415926535863945, axis 0.9999929999999873 9.234075398025226e-19 -0.0038130000033988177, limit lower=-0.523599 upper=0.523599 effort=60 velocity=100
- added joint Backpart_RR_j_hip: type revolute, parent Backpart, child RR_hip, origin xyz=-0.17626560000000002 -0.06932849 -0.0175 rpy=-1.5707963267948968 7.689375450873787e-28 -3.1415926535863945, axis 0.9999929999999873 9.234075398025226e-19 -0.0038130000033988177, limit lower=-0.523599 upper=0.523599 effort=60 velocity=100
- added joint Base_link_Back_j_Base: type revolute, parent Base_link, child Backpart, origin xyz=-0.18231475134396463 -0.165743138473793 0.29980299880961664 rpy=1.6528634893082283e-15 -5.094888957201467e-15 1.5746088781181597, axis 0.0 1.5706152165479998e-17 1.0, limit lower=-0.523599 upper=0.523599 effort=60 velocity=100
- added joint Base_link_Spine_j_Base: type revolute, parent Base_link, child Spine, origin xyz=-0.1753147504612079 -0.1657431406758344 0.29280299880961663 rpy=-1.5669837754716363 -1.5707963267948852 0, axis 1.5777107663893505e-30 0.999993 -0.003813, limit lower=-0.523599 upper=0.523599 effort=60 velocity=100
- added joint Frontpart_FL_j_hip: type revolute, parent Frontpart, child FL_hip, origin xyz=0.13877973000000002 0.01 0.0689438 rpy=3.1415926535897927 -4.771497806585007e-35 -3.944304526105059e-31, axis -0.999971 3.4020296938582826e-18 -0.007624999999996716, limit lower=-0.523599 upper=0.523599 effort=60 velocity=100
- added joint Frontpart_FR_j_hip: type revolute, parent Frontpart, child FR_hip, origin xyz=0.13771223 0.01 -0.07105213 rpy=3.1415926535897927 -4.771497806585007e-35 -3.944304526105059e-31, axis -0.999971 3.4020296938582826e-18 -0.007624999999996716, limit lower=-0.523599 upper=0.523599 effort=60 velocity=100
- added joint Spine_Front_j_Spine: type revolute, parent Spine, child Frontpart, origin xyz=0.0 -0.006633950000000004 0.04802529 rpy=1.5707963267948966 -1.5707963267948966 0, axis 0.999971 2.3476043000052282e-30 -0.007625, limit lower=-0.523599 upper=0.523599 effort=60 velocity=100
- joint FL_femur_FL_j_tibia: axis -7.888553831946753e-31 0.003812999999998753 0.999993 -> 0.0 0.999971 -0.0076249999999987534; limit (none) -> lower=-2.094395 upper=2.094395 effort=60 velocity=100; origin xyz=-0.13999999999999999 0.00021730999999991952 0.05699957999999999 rpy=-3.141592653589793 -7.8886090522100935e-31 -1.5777218104420243e-30 -> xyz=-0.13999999999999999 0.05699833999999998 -0.00043461999999983903 rpy=-3.141592653589793 1.5587779748584241e-43 -1.0097419586828949e-28; type continuous -> revolute
- joint FL_hip_FL_j_femur: axis 6.015853263215436e-33 0.0038129999999984574 0.9999930000000002 -> 1.0097126761660934e-28 0.9999710000000003 -0.0076249999999984585; limit (none) -> lower=-2.094395 upper=2.094395 effort=60 velocity=100; origin xyz=0.014221019999999812 3.552713678800501e-17 -0.057946209999999984 rpy=-1.5707963267948981 -4.461678287026247e-16 1.5707963267948966 -> xyz=0.05789157000000003 -3.552713678800501e-17 0.014441840000000004 rpy=-1.5707963267948981 -4.461678287026247e-16 1.5707963267948966; type continuous -> revolute
- joint FR_femur_FR_j_tibia: axis 7.888553831946753e-31 0.0038130000000016536 0.999993 -> 0.0 0.999971 -0.007625000000001654; limit (none) -> lower=-2.094395 upper=2.094395 effort=60 velocity=100; origin xyz=-0.13999999999999996 0.00021731000000009716 0.05699957999999999 rpy=-3.141592653589793 7.888609052210143e-31 1.577721810442022e-30 -> xyz=-0.14 0.05699833999999998 -0.0004346200000000522 rpy=-3.141592653589793 1.5570263517904096e-43 1.0097419586828949e-28; type continuous -> revolute
- joint FR_hip_FR_j_femur: axis -6.015853263215436e-33 0.0038130000000015435 0.9999930000000002 -> -1.0097126761660934e-28 0.9999710000000003 -0.007625000000001545; limit (none) -> lower=-2.094395 upper=2.094395 effort=60 velocity=100; origin xyz=-0.01377877000000021 3.552713678800501e-17 -0.05805294999999999 rpy=1.5707963267948981 -4.461678287026247e-16 1.5707963267948966 -> xyz=0.05810505999999993 0.0 -0.01355734000000001 rpy=1.5707963267948981 -4.461678287026247e-16 1.5707963267948966; type continuous -> revolute
- joint RL_femur_RL_j_tibia: axis -7.888553831946753e-31 0.003813000000001404 0.999993 -> 1.583726619652566e-30 0.9999930000000002 -0.0038130000000014055; limit (none) -> lower=-2.094395 upper=2.094395 effort=60 velocity=100; origin xyz=-0.13999999999999999 0.0002173200000000719 0.056999589999999996 rpy=-3.141592653589793 -0.0 0.0 -> xyz=-0.14 0.05699957999999998 -0.0002173100000000261 rpy=-3.141592653589793 -3.1554436208840465e-30 4.203895392974451e-45; type continuous -> revolute
- joint RL_hip_RL_j_femur: axis 7.888553831946753e-31 0.003813000000001293 0.999993 -> -1.5716949131261352e-30 0.9999930000000002 -0.0038130000000012945; limit (none) -> lower=-2.094395 upper=2.094395 effort=60 velocity=100; origin xyz=-0.013778779999802673 0.0 0.05805296000004681 rpy=-1.570796326798294 2.421734958835825e-16 -1.5707963267948966 -> xyz=0.0580529500000468 0.0 0.013778769999802693 rpy=-1.570796326798294 2.421734958835809e-16 -1.5707963267948966; type continuous -> revolute
- joint RR_femur_RR_j_tibia: axis 7.888553831946753e-31 0.003812999999998753 0.999993 -> -1.583726619652566e-30 0.9999930000000002 -0.003812999999998755; limit (none) -> lower=-2.094395 upper=2.094395 effort=60 velocity=100; origin xyz=-0.14 0.00021731999999985874 0.05699959000000001 rpy=-3.141592653589793 -0.0 0.0 -> xyz=-0.13999999999999999 0.056999589999999996 -0.00021731999999992978 rpy=-3.141592653589793 1.5777218104420233e-30 2.45227231256843e-45; type continuous -> revolute
- joint RR_hip_RR_j_femur: axis -7.888553831946753e-31 0.0038129999999984565 0.999993 -> 1.5777107663893505e-30 0.9999930000000002 -0.0038129999999984582; limit (none) -> lower=-2.094395 upper=2.094395 effort=60 velocity=100; origin xyz=0.014221030000196961 0.0 0.05794619999995167 rpy=1.5707963267914962 2.421734958835825e-16 -1.5707963267948966 -> xyz=0.05794619999995163 0.0 -0.014221030000196953 rpy=1.5707963267914962 2.421734958835809e-16 -1.5707963267948966; type continuous -> revolute
